Commit message: feat: :recycle: Mesh simplificado y ruedas radio normal

File: osr_gazebo/urdf/gazebo.urdf.xacro (robot description, xacro)
@@ -120,5 +120,5 @@
         <sensor name="imu_sensor" type="imu">
         <always_on>true</always_on>
-        <update_rate>100</update_rate>
+        <update_rate>10</update_rate>
         <visualize>true</visualize>
         <topic>"imu"</topic>
@@ -126,5 +126,5 @@
             <topicName>imu</topicName>
             <bodyName>imu_link</bodyName>
-            <updateRateHZ>100.0</updateRateHZ>
+            <updateRateHZ>50.0</updateRateHZ>
             <gaussianNoise>0.0</gaussianNoise>
             <xyzOffset>0 0 0</xyzOffset>

File: osr_gazebo/urdf/osr_mod.urdf.xacro (robot description, xacro)
@@ -23,5 +23,5 @@
             <origin rpy="0 0 0" xyz="0 0 0.0"/>
             <geometry>
-                <mesh filename="file://$(find osr_gazebo)/meshes/body.stl"/>
+                <mesh filename="file://$(find osr_gazebo)/simple_meshes/body.stl"/>
             </geometry>
         </collision>
@@ -29,5 +29,5 @@
             <origin rpy="0 0 0" xyz="0 0 0.0"/>
             <geometry>
-                <mesh filename="file://$(find osr_gazebo)/meshes/body.stl"/>
+                <mesh filename="file://$(find osr_gazebo)/simple_meshes/body.stl"/>
             </geometry>
             <material name="brown"/>
@@ -49,5 +49,5 @@
             <origin rpy="0 0 -3.14" xyz="0 0 0.0"/>
             <geometry>
-                <mesh filename="file://$(find osr_gazebo)/meshes/box_link.stl"/>
+                <mesh filename="file://$(find osr_gazebo)/simple_meshes/box_link.stl"/>
             </geometry>
         </collision>
@@ -55,5 +55,5 @@
             <origin rpy="0 0 -3.14" xyz="0 0 0"/>
             <geometry>
-                <mesh filename="file://$(find osr_gazebo)/meshes/box_link.stl"/>
+                <mesh filename="file://$(find osr_gazebo)/simple_meshes/box_link.stl"/>
             </geometry>
             <material name="silver"/>
@@ -76,5 +76,5 @@
                 <origin rpy="0 0.2 0" xyz="0 0 0"/>
                 <geometry>
-                    <mesh filename="file://$(find osr_gazebo)/meshes/arm.stl"/>
+                    <mesh filename="file://$(find osr_gazebo)/simple_meshes/arm.stl"/>
                 </geometry>
             </collision>
@@ -82,5 +82,5 @@
                 <origin rpy="0 0.2 0" xyz="0 0 0"/>
                 <geometry>
-                    <mesh filename="file://$(find osr_gazebo)/meshes/arm.stl"/>
+                    <mesh filename="file://$(find osr_gazebo)/simple_meshes/arm.stl"/>
                 </geometry>
                 <material name="silver"/>
@@ -106,5 +106,5 @@
                 <origin rpy="0 0 ${origin}" xyz="0 0 0.0"/>
                 <geometry>
-                    <mesh filename="file://$(find osr_gazebo)/meshes/turn_${prefix}.stl"/>
+                    <mesh filename="file://$(find osr_gazebo)/simple_meshes/turn_${prefix}.stl"/>
                 </geometry>
             </collision>
@@ -112,5 +112,5 @@
                 <origin rpy="0 0 ${origin}" xyz="0 0 0.0"/>
                 <geometry>
-                    <mesh filename="file://$(find osr_gazebo)/meshes/turn_${prefix}.stl"/>
+                    <mesh filename="file://$(find osr_gazebo)/simple_meshes/turn_${prefix}.stl"/>
                 </geometry>
                 <material name="silver"/>
@@ -136,5 +136,5 @@
                 <origin rpy="0 0 1.57" xyz="0 0 0.0"/>
                 <geometry>
-                    <mesh filename="file://$(find osr_gazebo)/meshes/body_axis.stl"/>
+                    <mesh filename="file://$(find osr_gazebo)/simple_meshes/body_axis.stl"/>
                 </geometry>
             </collision>
@@ -142,5 +142,5 @@
                 <origin rpy="0 0 1.57" xyz="0 0 0.0"/>
                 <geometry>
-                    <mesh filename="file://$(find osr_gazebo)/meshes/body_axis.stl"/>
+                    <mesh filename="file://$(find osr_gazebo)/simple_meshes/body_axis.stl"/>
                 </geometry>
                 <material name="silver"/>
@@ -166,11 +166,11 @@
                 <origin rpy="0 0 0" xyz="0 0 0.0"/>
                 <geometry>
-                    <mesh filename="file://$(find osr_gazebo)/meshes/rockerbogie_middle_1.stl"/>
-                </geometry>
-            </collision>
-            <visual>
-                <origin rpy="0 0 0" xyz="0 0 0.0"/>
-                <geometry>
-                    <mesh filename="file://$(find osr_gazebo)/meshes/rockerbogie_middle_1.stl"/>
+                    <mesh filename="file://$(find osr_gazebo)/simple_meshes/rockerbogie_middle_1.stl"/>
+                </geometry>
+            </collision>
+            <visual>
+                <origin rpy="0 0 0" xyz="0 0 0.0"/>
+                <geometry>
+                    <mesh filename="file://$(find osr_gazebo)/simple_meshes/rockerbogie_middle_1.stl"/>
                 </geometry>
                 <material name="silver"/>
@@ -193,11 +193,11 @@
                 <origin rpy="0 0 0" xyz="0 0 0.0"/>
                 <geometry>
-                    <mesh filename="file://$(find osr_gazebo)/meshes/rockerbogie_front_1.stl"/>
-                </geometry>
-            </collision>
-            <visual>
-                <origin rpy="0 0 0" xyz="0 0 0.0"/>
-                <geometry>
-                    <mesh filename="file://$(find osr_gazebo)/meshes/rockerbogie_front_1.stl"/>
+                    <mesh filename="file://$(find osr_gazebo)/simple_meshes/rockerbogie_front_1.stl"/>
+                </geometry>
+            </collision>
+            <visual>
+                <origin rpy="0 0 0" xyz="0 0 0.0"/>
+                <geometry>
+                    <mesh filename="file://$(find osr_gazebo)/simple_meshes/rockerbogie_front_1.stl"/>
                 </geometry>
                 <material name="silver"/>
@@ -224,5 +224,5 @@
                 <origin rpy="0 0 ${dir*-1.57}" xyz="0 0 0.0"/>
                 <geometry>
-                    <mesh filename="file://$(find osr_gazebo)/meshes/wheel_link_left_2.stl"/>
+                    <mesh filename="file://$(find osr_gazebo)/simple_meshes/wheel_link_left_2.stl"/>
                 </geometry>
             </collision>
@@ -230,5 +230,5 @@
                 <origin rpy="0 0 ${dir*-1.57}" xyz="0 0 0.0"/>
                 <geometry>
-                    <mesh filename="file://$(find osr_gazebo)/meshes/wheel_link_left_2.stl"/>
+                    <mesh filename="file://$(find osr_gazebo)/simple_meshes/wheel_link_left_2.stl"/>
                 </geometry>
                 <material name="silver"/>
@@ -252,5 +252,6 @@
                 <origin rpy="${origin} 0 ${-dir*1.57}" xyz="0 0 0.0"/>
                 <geometry>
-                    <mesh filename="file://$(find osr_gazebo)/meshes/wheel_middle_left.stl"/>
+                    <!-- <cylinder radius="0.03" length="0.04"/> -->
+                    <mesh filename="file://$(find osr_gazebo)/simple_meshes/wheel_middle_left.stl"/>
                 </geometry>
             </collision>
@@ -258,5 +259,6 @@
                 <origin rpy="${origin} 0 ${-dir*1.57}" xyz="0 0 0.0"/>
                 <geometry>
-                    <mesh filename="file://$(find osr_gazebo)/meshes/wheel_middle_left.stl"/>
+                    <!-- <cylinder radius="0.03" length="0.04"/> -->
+                    <mesh filename="file://$(find osr_gazebo)/simple_meshes/wheel_middle_left.stl"/>
                 </geometry>
                 <material name="silver"/>
@@ -278,5 +280,6 @@
                 <origin rpy="0 0 ${-dir*1.57}" xyz="0 0 0.0"/>
                 <geometry>
-                    <mesh filename="file://$(find osr_gazebo)/meshes/wheel_link_left_2.stl"/>
+                    <!-- <cylinder radius="0.03" length="0.04"/> -->
+                    <mesh filename="file://$(find osr_gazebo)/simple_meshes/wheel_link_left_2.stl"/>
                 </geometry>
             </collision>
@@ -284,5 +287,6 @@
                 <origin rpy="0 0 ${-dir*1.57}" xyz="0 0 0.0"/>
                 <geometry>
-                    <mesh filename="file://$(find osr_gazebo)/meshes/wheel_link_left_2.stl"/>
+                    <!-- <cylinder radius="0.03" length="0.04"/> -->
+                    <mesh filename="file://$(find osr_gazebo)/simple_meshes/wheel_link_left_2.stl"/>
                 </geometry>
                 <material name="silver"/>
@@ -310,5 +314,6 @@
                 <origin rpy="-1.57 0 ${origin}" xyz="0 0 0.0"/>
                 <geometry>
-                    <mesh filename="file://$(find osr_gazebo)/meshes/wheel.stl"/>
+                    <cylinder radius="0.082" length="0.04"/>
+                    <!-- <mesh filename="file://$(find osr_gazebo)/simple_meshes/wheel.stl"/> -->
                 </geometry>
                 <surface>
@@ -324,5 +329,6 @@
                 <origin rpy="-1.57 0 ${origin}" xyz="0 0 0.0"/>
                 <geometry>
-                    <mesh filename="file://$(find osr_gazebo)/meshes/wheel.stl"/>
+                    <cylinder radius="0.082" length="0.04"/>
+                    <!-- <mesh filename="file://$(find osr_gazebo)/simple_meshes/wheel.stl"/> -->
                 </geometry>
                 <material name="black"/>
@@ -345,5 +351,6 @@
                 <origin rpy="-1.57 0 ${origin}" xyz="0 0 0.0"/>
                 <geometry>
-                    <mesh filename="file://$(find osr_gazebo)/meshes/wheel.stl"/>
+                    <cylinder radius="0.082" length="0.04"/>
+                    <!-- <mesh filename="file://$(find osr_gazebo)/simple_meshes/wheel.stl"/> -->
                 </geometry>
                 <surface>
@@ -359,5 +366,6 @@
                 <origin rpy="-1.57 0 ${origin}" xyz="0 0 0.0"/>
                 <geometry>
-                    <mesh filename="file://$(find osr_gazebo)/meshes/wheel.stl"/>
+                    <cylinder radius="0.082" length="0.04"/>
+                    <!-- <mesh filename="file://$(find osr_gazebo)/simple_meshes/wheel.stl"/> -->
                 </geometry>
                 <material name="black"/>
@@ -380,5 +388,6 @@
                 <origin rpy="-1.57 0 ${origin}" xyz="0 0 0.0"/>
                 <geometry>
-                    <mesh filename="file://$(find osr_gazebo)/meshes/wheel.stl"/>
+                    <cylinder radius="0.082" length="0.04"/>
+                    <!-- <mesh filename="file://$(find osr_gazebo)/simple_meshes/wheel.stl"/> -->
                 </geometry>
                 <surface>
@@ -394,5 +403,6 @@
                 <origin rpy="-1.57 0 ${origin}" xyz="0 0 0.0"/>
                 <geometry>
-                    <mesh filename="file://$(find osr_gazebo)/meshes/wheel.stl"/>
+                    <cylinder radius="0.082" length="0.04"/>
+                    <!-- <mesh filename="file://$(find osr_gazebo)/simple_meshes/wheel.stl"/> -->
                 </geometry>
                 <material name="black"/>
